Commit message: 101: joint, base to sub

File: bot101.urdf (robot description, URDF)
Before this commit: robot bot101, 1 links, 0 joints
Links:
- added link sub_link, mass 0.25; collision cylinder length=1 radius=0.1; visual cylinder length=1 radius=0.1
Joints:
- added joint base_to_sub: type fixed, parent base_link, child sub_link, origin xyz=0.5 0 0 rpy=0 0 0, axis 1 0 0, limit lower=10 upper=0 effort=10 velocity=1

Commit message: joint: moving now

File: bot101.urdf (robot description, URDF)
Before this commit: robot bot101, 2 links, 1 joints
Joints:
- joint base_to_sub: type fixed -> revolute

Commit message: bots are moving!

File: bot101.urdf (robot description, URDF)
Before this commit: robot bot101, 2 links, 1 joints
Links:
- added link sub_link_2, mass 0.25; collision cylinder length=2 radius=0.05; visual cylinder length=2 radius=0.05
Joints:
- added joint base_to_sub_2: type revolute, parent base_link, child sub_link_2, origin xyz=1 0 0 rpy=0 0 0, axis 1 0 0, limit lower=10 upper=0 effort=10 velocity=1
